File: hardware/rfboard.sch (KiCad schematic (older format))
At the start: 20 parts, among them J1 10118194-0001LF, P2 CONN_01X03, P3 CONN_01X04, P5 CONN_01X01, U1 SAMD21E18, U2 RFM69CW-915MHZ, U3 MIC5504-3.3YM5-T5

Commit message: Associate footprints
Parts:
- C1, C2: value C -> 1uF; footprint (none) -> Capacitors_SMD:C_0603_HandSoldering
- C3: value C -> 10uF; footprint (none) -> Capacitors_SMD:C_0805_HandSoldering
- D2: footprint (none) -> LEDs:LED_0603
- H1, H2, H3: footprint (none) -> Mounting_Holes:MountingHole_2.7mm_M2.5_Pad
- J2, J3: renamed from J?; footprint (none) -> Pin_Headers:Pin_Header_Straight_1x11_Pitch2.54mm
- P2: footprint SparkFun-Connectors:1X03 -> Sparkfun-Connectors:1X03
- P3: footprint SparkFun-Connectors:1X04 -> Sparkfun-Connectors:1X04
- P5: footprint SparkFun-Connectors:1X01 -> Sparkfun-Connectors:1X01
- R1: footprint SparkFun-Resistors:0603 -> Resistors_SMD:R_0603_HandSoldering
- R2: footprint (none) -> Resistors_SMD:R_0603_HandSoldering
- R3: renamed from R?; footprint (none) -> Resistors_SMD:R_0603_HandSoldering
- U1: footprint (none) -> Sparkfun-Silicon-Standard:TQFP32-08
- U2: footprint RFM69CW-XXXS2 -> homebrew:RFM69CW-XXXS2_
- U3: footprint SOT23-5P95_280X145XL45X37N -> MIC5504-3.3YM5-T5:SOT23-5P95_280X145XL45X37N
Changed lines of the file:
@@
 F 0 "P2" H 2850 7650 50  0000 C CNN
 F 1 "CONN_01X03" V 2950 7450 50  0000 C CNN
-F 2 "SparkFun-Connectors:1X03" H 2850 7450 50  0001 C CNN
+F 2 "Sparkfun-Connectors:1X03" H 2850 7450 50  0001 C CNN
 F 3 "" H 2850 7450 50  0000 C CNN
 	1    2850 7450
@@
 F 0 "P3" H 3750 7650 50  0000 C CNN
 F 1 "CONN_01X04" V 3850 7400 50  0000 C CNN
-F 2 "SparkFun-Connectors:1X04" H 3750 7400 50  0001 C CNN
+F 2 "Sparkfun-Connectors:1X04" H 3750 7400 50  0001 C CNN
 F 3 "" H 3750 7400 50  0000 C CNN
 	1    3750 7400
@@
 F 0 "P5" H 5000 7500 50  0000 C CNN
 F 1 "CONN_01X01" V 5100 7400 50  0000 C CNN
-F 2 "SparkFun-Connectors:1X01" H 5000 7400 50  0001 C CNN
+F 2 "Sparkfun-Connectors:1X01" H 5000 7400 50  0001 C CNN
 F 3 "" H 5000 7400 50  0000 C CNN
 	1    5000 7400
@@
 F 0 "R1" V 8280 850 50  0000 C CNN
 F 1 "220" V 8200 850 50  0000 C CNN
-F 2 "SparkFun-Resistors:0603" V 8130 850 50  0001 C CNN
+F 2 "Resistors_SMD:R_0603_HandSoldering" V 8130 850 50  0001 C CNN
 F 3 "" H 8200 850 50  0000 C CNN
 	1    8200 850
@@
 F 0 "U2" H 4500 2250 45  0000 L BNN
 F 1 "RFM69CW-915MHZ" H 4500 1100 45  0000 L BNN
-F 2 "RFM69CW-XXXS2" H 4900 2300 20  0001 C CNN
+F 2 "homebrew:RFM69CW-XXXS2_" H 4900 2300 20  0001 C CNN
 F 3 "" H 4900 1700 60  0001 C CNN
 F 4 "IC-11996" H 4900 2350 60  0000 C CNN "Field4"
@@
 F 0 "H1" H 6100 6570 60  0000 C CNN
 F 1 "HOLE" H 6100 6820 60  0000 C CNN
-F 2 "" H 6100 6700 60  0001 C CNN
+F 2 "Mounting_Holes:MountingHole_2.7mm_M2.5_Pad" H 6100 6700 60  0001 C CNN
 F 3 "" H 6100 6700 60  0001 C CNN
 	1    6100 6700
@@
 F 0 "H2" H 6100 6970 60  0000 C CNN
 F 1 "HOLE" H 6100 7220 60  0000 C CNN
-F 2 "" H 6100 7100 60  0001 C CNN
+F 2 "Mounting_Holes:MountingHole_2.7mm_M2.5_Pad" H 6100 7100 60  0001 C CNN
 F 3 "" H 6100 7100 60  0001 C CNN
 	1    6100 7100
@@
 F 0 "H3" H 6100 7370 60  0000 C CNN
 F 1 "HOLE" H 6100 7620 60  0000 C CNN
-F 2 "" H 6100 7500 60  0001 C CNN
+F 2 "Mounting_Holes:MountingHole_2.7mm_M2.5_Pad" H 6100 7500 60  0001 C CNN
 F 3 "" H 6100 7500 60  0001 C CNN
 	1    6100 7500
@@
 F 0 "U3" H 9549 1271 50  0000 L BNN
 F 1 "MIC5504-3.3YM5-T5" H 9350 550 50  0000 L BNN
-F 2 "SOT23-5P95_280X145XL45X37N" H 9850 950 50  0001 L BNN
+F 2 "MIC5504-3.3YM5-T5:SOT23-5P95_280X145XL45X37N" H 9850 950 50  0001 L BNN
 F 3 "Microchip" H 9850 950 50  0001 L BNN
 F 4 "SOT-23-5 Microchip" H 9850 950 50  0001 L BNN "Field4"
@@
 P 10500 1000
 F 0 "C1" H 10525 1100 50  0000 L CNN
-F 1 "C" H 10525 900 50  0000 L CNN
-F 2 "" H 10538 850 50  0001 C CNN
+F 1 "1uF" H 10525 900 50  0000 L CNN
+F 2 "Capacitors_SMD:C_0603_HandSoldering" H 10538 850 50  0001 C CNN
 F 3 "" H 10500 1000 50  0001 C CNN
 	1    10500 1000
@@
 P 10750 1000
 F 0 "C2" H 10775 1100 50  0000 L CNN
-F 1 "C" H 10775 900 50  0000 L CNN
-F 2 "" H 10788 850 50  0001 C CNN
+F 1 "1uF" H 10775 900 50  0000 L CNN
+F 2 "Capacitors_SMD:C_0603_HandSoldering" H 10788 850 50  0001 C CNN
 F 3 "" H 10750 1000 50  0001 C CNN
 	1    10750 1000
@@
 P 11000 1000
 F 0 "C3" H 11025 1100 50  0000 L CNN
-F 1 "C" H 11025 900 50  0000 L CNN
-F 2 "" H 11038 850 50  0001 C CNN
+F 1 "10uF" H 11025 900 50  0000 L CNN
+F 2 "Capacitors_SMD:C_0805_HandSoldering" H 11038 850 50  0001 C CNN
 F 3 "" H 11000 1000 50  0001 C CNN
 	1    11000 1000
@@
 F 0 "U1" H 1650 700 60  0000 C CNN
 F 1 "SAMD21E18" H 1650 3400 60  0000 C CNN
-F 2 "" H 1750 2150 60  0001 C CNN
+F 2 "Sparkfun-Silicon-Standard:TQFP32-08" H 1750 2150 60  0001 C CNN
 F 3 "" H 1750 2150 60  0001 C CNN
 	1    1750 2150
@@
 F 0 "D2" H 7450 2000 50  0000 C CNN
 F 1 "LED" H 7450 1800 50  0000 C CNN
-F 2 "" H 7450 1900 50  0001 C CNN
+F 2 "LEDs:LED_0603" H 7450 1900 50  0001 C CNN
 F 3 "" H 7450 1900 50  0001 C CNN
 	1    7450 1900
@@
 F 0 "R2" V 7230 1900 50  0000 C CNN
 F 1 "1k" V 7150 1900 50  0000 C CNN
-F 2 "" V 7080 1900 50  0001 C CNN
+F 2 "Resistors_SMD:R_0603_HandSoldering" V 7080 1900 50  0001 C CNN
 F 3 "" H 7150 1900 50  0001 C CNN
 	1    7150 1900
@@
 NoConn ~ 1100 1300
 $Comp
-L CONN_01X11 J?
+L CONN_01X11 J2
 U 1 1 5A857114
 P 10550 2450
-F 0 "J?" H 10550 3050 50  0000 C CNN
+F 0 "J2" H 10550 3050 50  0000 C CNN
 F 1 "CONN_01X11" V 10650 2450 50  0000 C CNN
-F 2 "" H 10550 2450 50  0001 C CNN
+F 2 "Pin_Headers:Pin_Header_Straight_1x11_Pitch2.54mm" H 10550 2450 50  0001 C CNN
 F 3 "" H 10550 2450 50  0001 C CNN
 	1    10550 2450
@@
 $EndComp
 $Comp
-L CONN_01X11 J?
+L CONN_01X11 J3
 U 1 1 5A8571EF
 P 10550 3750
-F 0 "J?" H 10550 4350 50  0000 C CNN
+F 0 "J3" H 10550 4350 50  0000 C CNN
 F 1 "CONN_01X11" V 10650 3750 50  0000 C CNN
-F 2 "" H 10550 3750 50  0001 C CNN
+F 2 "Pin_Headers:Pin_Header_Straight_1x11_Pitch2.54mm" H 10550 3750 50  0001 C CNN
 F 3 "" H 10550 3750 50  0001 C CNN
 	1    10550 3750
@@
 $EndComp
 $Comp
-L GND #PWR?
+L GND #PWR019
 U 1 1 5A857326
-P 10350 4300
-F 0 "#PWR?" H 10350 4050 50  0001 C CNN
-F 1 "GND" H 10350 4150 50  0000 C CNN
-F 2 "" H 10350 4300 50  0001 C CNN
-F 3 "" H 10350 4300 50  0001 C CNN
-	1    10350 4300
-	1    0    0    -1
-$EndComp
-$Comp
-L GND #PWR?
+P 10350 4250
+F 0 "#PWR019" H 10350 4000 50  0001 C CNN
+F 1 "GND" H 10350 4100 50  0000 C CNN
+F 2 "" H 10350 4250 50  0001 C CNN
+F 3 "" H 10350 4250 50  0001 C CNN
+	1    10350 4250
+	1    0    0    -1
+$EndComp
+$Comp
+L GND #PWR020
 U 1 1 5A857360
 P 10350 2950
-F 0 "#PWR?" H 10350 2700 50  0001 C CNN
+F 0 "#PWR020" H 10350 2700 50  0001 C CNN
 F 1 "GND" H 10350 2800 50  0000 C CNN
 F 2 "" H 10350 2950 50  0001 C CNN
@@
 $EndComp
 $Comp
-L +3V3 #PWR?
+L +3V3 #PWR021
 U 1 1 5A85739A
 P 9550 4150
-F 0 "#PWR?" H 9550 4000 50  0001 C CNN
+F 0 "#PWR021" H 9550 4000 50  0001 C CNN
 F 1 "+3V3" H 9550 4290 50  0000 C CNN
 F 2 "" H 9550 4150 50  0001 C CNN
@@
 $EndComp
 $Comp
-L +3V3 #PWR?
+L +3V3 #PWR022
 U 1 1 5A8574DE
 P 9500 2850
-F 0 "#PWR?" H 9500 2700 50  0001 C CNN
+F 0 "#PWR022" H 9500 2700 50  0001 C CNN
 F 1 "+3V3" H 9500 2990 50  0000 C CNN
 F 2 "" H 9500 2850 50  0001 C CNN
@@
 $EndComp
 $Comp
-L +5V #PWR?
+L +5V #PWR023
 U 1 1 5A85766A
 P 9700 4050
-F 0 "#PWR?" H 9700 3900 50  0001 C CNN
+F 0 "#PWR023" H 9700 3900 50  0001 C CNN
 F 1 "+5V" H 9700 4190 50  0000 C CNN
 F 2 "" H 9700 4050 50  0001 C CNN
@@
 $EndComp
 $Comp
-L +5V #PWR?
+L +5V #PWR024
 U 1 1 5A857833
 P 9650 2750
-F 0 "#PWR?" H 9650 2600 50  0001 C CNN
+F 0 "#PWR024" H 9650 2600 50  0001 C CNN
 F 1 "+5V" H 9650 2890 50  0000 C CNN
 F 2 "" H 9650 2750 50  0001 C CNN
@@
 LED_EXTERNAL_2
 $Comp
-L R R?
+L R R3
 U 1 1 5A858695
 P 10200 1950
-F 0 "R?" V 10280 1950 50  0000 C CNN
+F 0 "R3" V 10280 1950 50  0000 C CNN
 F 1 "220" V 10200 1950 50  0000 C CNN
-F 2 "" V 10130 1950 50  0001 C CNN
+F 2 "Resistors_SMD:R_0603_HandSoldering" V 10130 1950 50  0001 C CNN
 F 3 "" H 10200 1950 50  0001 C CNN
 	1    10200 1950

Commit message: Layed out the components.
Parts:
- H1, H2, H3: footprint Mounting_Holes:MountingHole_2.7mm_M2.5_Pad -> homebrew:MountingHole_2.7mm_M2.5
Changed lines of the file:
@@
 F 0 "H1" H 6100 6570 60  0000 C CNN
 F 1 "HOLE" H 6100 6820 60  0000 C CNN
-F 2 "Mounting_Holes:MountingHole_2.7mm_M2.5_Pad" H 6100 6700 60  0001 C CNN
+F 2 "homebrew:MountingHole_2.7mm_M2.5" H 6100 6700 60  0001 C CNN
 F 3 "" H 6100 6700 60  0001 C CNN
 	1    6100 6700
@@
 F 0 "H2" H 6100 6970 60  0000 C CNN
 F 1 "HOLE" H 6100 7220 60  0000 C CNN
-F 2 "Mounting_Holes:MountingHole_2.7mm_M2.5_Pad" H 6100 7100 60  0001 C CNN
+F 2 "homebrew:MountingHole_2.7mm_M2.5" H 6100 7100 60  0001 C CNN
 F 3 "" H 6100 7100 60  0001 C CNN
 	1    6100 7100
@@
 F 0 "H3" H 6100 7370 60  0000 C CNN
 F 1 "HOLE" H 6100 7620 60  0000 C CNN
-F 2 "Mounting_Holes:MountingHole_2.7mm_M2.5_Pad" H 6100 7500 60  0001 C CNN
+F 2 "homebrew:MountingHole_2.7mm_M2.5" H 6100 7500 60  0001 C CNN
 F 3 "" H 6100 7500 60  0001 C CNN
 	1    6100 7500

Commit message: Finished layout.
Connections:
- net labels added: L1, L2, L3, L4, L5, L6, R1, R2, R3, R4, R5, R6, R7, R8
- wire segments 18 -> 19
Changed lines of the file:
@@
 	0    1    1    0
 $EndComp
+Text GLabel 10350 2050 0    60   Input ~ 0
+L1
+Text GLabel 10350 2150 0    60   Input ~ 0
+L2
+Text GLabel 10350 2250 0    60   Input ~ 0
+L3
+Text GLabel 10350 2350 0    60   Input ~ 0
+L4
+Text GLabel 10350 2450 0    60   Input ~ 0
+L5
+Text GLabel 10350 2550 0    60   Input ~ 0
+L6
+Text GLabel 10350 3250 0    60   Input ~ 0
+R1
+Text GLabel 10350 3350 0    60   Input ~ 0
+R2
+Text GLabel 10350 3450 0    60   Input ~ 0
+R3
+Text GLabel 10350 3550 0    60   Input ~ 0
+R4
+Text GLabel 10350 3650 0    60   Input ~ 0
+R5
+Text GLabel 10350 3750 0    60   Input ~ 0
+R6
+Text GLabel 10350 3850 0    60   Input ~ 0
+R7
+Text GLabel 10350 3950 0    60   Input ~ 0
+R8
+Text GLabel 2200 1500 2    60   Input ~ 0
+R8
+Text GLabel 2200 1400 2    60   Input ~ 0
+R7
+Text GLabel 2200 1300 2    60   Input ~ 0
+R6
+Text GLabel 2200 1200 2    60   Input ~ 0
+R5
+Text GLabel 2200 1100 2    60   Input ~ 0
+R4
+Text GLabel 2200 1000 2    60   Input ~ 0
+R3
+Text GLabel 2200 2900 2    60   Input ~ 0
+R2
+Text GLabel 2200 2800 2    60   Input ~ 0
+R1
+Text GLabel 2200 2700 2    60   Input ~ 0
+L1
+Text GLabel 2200 2600 2    60   Input ~ 0
+L2
+Text GLabel 2200 2500 2    60   Input ~ 0
+L3
+Text GLabel 2200 2400 2    60   Input ~ 0
+L4
+Text GLabel 2200 2300 2    60   Input ~ 0
+L5
+Text GLabel 2200 2200 2    60   Input ~ 0
+L6
+$Comp
+L +5V #PWR?
+U 1 1 5A867DF0
+P 9800 2650
+F 0 "#PWR?" H 9800 2500 50  0001 C CNN
+F 1 "+5V" H 9800 2790 50  0000 C CNN
+F 2 "" H 9800 2650 50  0001 C CNN
+F 3 "" H 9800 2650 50  0001 C CNN
+	1    9800 2650
+	1    0    0    -1
+$EndComp
+Wire Wire Line
+	9800 2650 10350 2650
 $EndSCHEMATC
