File: hardware/rfboard.sch (KiCad schematic (older format))
At the start: 20 parts, among them J1 10118194-0001LF, J2 Conn_01x10, J3 Conn_01x10, P2 CONN_01X03, P3 CONN_01X04, P5 CONN_01X01, U1 SAMD21E18, U2 RFM69CW-915MHZ, U3 MIC5504-3.3YM5-T5, U4 74LVC1G125

Commit message: Hardware revision 1.2:
- Add pullup resistors for doing I2C
- Added a helical antenna (untested)
Parts:
- removed P5: CONN_01X01, Pin_Headers:Pin_Header_Straight_1x01_Pitch2.54mm, symbol CONN_01X01
- added AE1: Antenna, homebrew:helical_antenna_915mhz_hole, symbol Antenna
- added R1, R3: 4k7, Resistors_SMD:R_0603, symbol R
Connections:
- net labels added: SCL, SDA
- net labels removed: R1, R2
- wire segments 25 -> 32
Other:
- moved on the sheet: J3
Changed lines of the file:
@@
-	1    0    0    -1
-$EndComp
-$Comp
-L CONN_01X01 P5
-U 1 1 5A542715
-P 5000 7400
-F 0 "P5" H 5000 7500 50  0000 C CNN
-F 1 "CONN_01X01" V 5100 7400 50  0000 C CNN
-F 2 "Pin_Headers:Pin_Header_Straight_1x01_Pitch2.54mm" H 5000 7400 50  0001 C CNN
-F 3 "" H 5000 7400 50  0000 C CNN
-	1    5000 7400
 	1    0    0    -1
 $EndComp
@@
 L GND #PWR018
 U 1 1 5A857326
-P 10350 4250
-F 0 "#PWR018" H 10350 4000 50  0001 C CNN
-F 1 "GND" H 10350 4100 50  0000 C CNN
-F 2 "" H 10350 4250 50  0001 C CNN
-F 3 "" H 10350 4250 50  0001 C CNN
-	1    10350 4250
+P 10350 4850
+F 0 "#PWR018" H 10350 4600 50  0001 C CNN
+F 1 "GND" H 10350 4700 50  0000 C CNN
+F 2 "" H 10350 4850 50  0001 C CNN
+F 3 "" H 10350 4850 50  0001 C CNN
+	1    10350 4850
 	1    0    0    -1
 $EndComp
@@
 L +3V3 #PWR020
 U 1 1 5A85739A
-P 9550 4050
-F 0 "#PWR020" H 9550 3900 50  0001 C CNN
-F 1 "+3V3" H 9550 4190 50  0000 C CNN
-F 2 "" H 9550 4050 50  0001 C CNN
-F 3 "" H 9550 4050 50  0001 C CNN
-	1    9550 4050
+P 9550 4650
+F 0 "#PWR020" H 9550 4500 50  0001 C CNN
+F 1 "+3V3" H 9550 4790 50  0000 C CNN
+F 2 "" H 9550 4650 50  0001 C CNN
+F 3 "" H 9550 4650 50  0001 C CNN
+	1    9550 4650
 	1    0    0    -1
 $EndComp
@@
 L +5V #PWR022
 U 1 1 5A85766A
-P 9700 3950
-F 0 "#PWR022" H 9700 3800 50  0001 C CNN
-F 1 "+5V" H 9700 4090 50  0000 C CNN
-F 2 "" H 9700 3950 50  0001 C CNN
-F 3 "" H 9700 3950 50  0001 C CNN
-	1    9700 3950
+P 9700 4550
+F 0 "#PWR022" H 9700 4400 50  0001 C CNN
+F 1 "+5V" H 9700 4690 50  0000 C CNN
+F 2 "" H 9700 4550 50  0001 C CNN
+F 3 "" H 9700 4550 50  0001 C CNN
+	1    9700 4550
 	1    0    0    -1
 $EndComp
@@
 Text GLabel 10350 2550 0    60   Input ~ 0
 L6
-Text GLabel 10350 3350 0    60   Input ~ 0
-R1
-Text GLabel 10350 3450 0    60   Input ~ 0
-R2
-Text GLabel 10350 3550 0    60   Input ~ 0
+Text GLabel 10200 3950 0    60   Input ~ 0
+SDA
+Text GLabel 10300 4050 0    60   Input ~ 0
+SCL
+Text GLabel 10350 4150 0    60   Input ~ 0
 R3
-Text GLabel 10350 3650 0    60   Input ~ 0
+Text GLabel 10350 4250 0    60   Input ~ 0
 R4
-Text GLabel 10350 3750 0    60   Input ~ 0
+Text GLabel 10350 4350 0    60   Input ~ 0
 R5
-Text GLabel 10350 3850 0    60   Input ~ 0
+Text GLabel 10350 4450 0    60   Input ~ 0
 R6
 Text GLabel 2200 1500 2    60   Input ~ 0
@@
 R3
 Text GLabel 2200 2900 2    60   Input ~ 0
-R2
+SCL
 Text GLabel 2200 2800 2    60   Input ~ 0
-R1
+SDA
 Text GLabel 2200 2700 2    60   Input ~ 0
 L1
@@
 	10350 2750 9650 2750
 Wire Wire Line
-	10350 4050 9550 4050
-Wire Wire Line
-	9700 3950 10350 3950
+	10350 4650 9550 4650
+Wire Wire Line
+	9700 4550 10350 4550
 Wire Wire Line
 	9800 2650 10350 2650
@@
 	1300 5550 1300 5450
 Wire Wire Line
-	1300 5450 1350 5450
-Wire Wire Line
-	1350 5450 1400 5450
+	1300 5450 1400 5450
 Text GLabel 1800 5450 2    60   Input ~ 0
 RESET_SW
@@
 L Conn_01x10 J3
 U 1 1 5B41AA32
-P 10550 3750
-F 0 "J3" H 10550 4250 50  0000 C CNN
-F 1 "Conn_01x10" H 10550 3150 50  0000 C CNN
-F 2 "Pin_Headers:Pin_Header_Straight_1x10_Pitch2.54mm" H 10550 3750 50  0001 C CNN
-F 3 "" H 10550 3750 50  0001 C CNN
-	1    10550 3750
-	1    0    0    -1
-$EndComp
-Wire Wire Line
-	10350 4150 10350 4250
+P 10550 4350
+F 0 "J3" H 10550 4850 50  0000 C CNN
+F 1 "Conn_01x10" H 10550 3750 50  0000 C CNN
+F 2 "Pin_Headers:Pin_Header_Straight_1x10_Pitch2.54mm" H 10550 4350 50  0001 C CNN
+F 3 "" H 10550 4350 50  0001 C CNN
+	1    10550 4350
+	1    0    0    -1
+$EndComp
+Wire Wire Line
+	10350 4750 10350 4850
 $Comp
 L MOMENTARY-SWITCH-SPST-SMD-4.6X2.8MM S1
@@
 	1    0    0    -1
 $EndComp
+Wire Wire Line
+	10200 3950 10350 3950
+Wire Wire Line
+	10300 4050 10350 4050
+$Comp
+L +3V3 #PWR030
+U 1 1 5C7E03DA
+P 10350 3550
+F 0 "#PWR030" H 10350 3400 50  0001 C CNN
+F 1 "+3V3" H 10350 3690 50  0000 C CNN
+F 2 "" H 10350 3550 50  0001 C CNN
+F 3 "" H 10350 3550 50  0001 C CNN
+	1    10350 3550
+	1    0    0    -1
+$EndComp
+$Comp
+L R R3
+U 1 1 5C7E05DB
+P 10350 3750
+F 0 "R3" V 10430 3750 50  0000 C CNN
+F 1 "4k7" V 10350 3750 50  0000 C CNN
+F 2 "Resistors_SMD:R_0603" V 10280 3750 50  0001 C CNN
+F 3 "" H 10350 3750 50  0001 C CNN
+	1    10350 3750
+	-1   0    0    1
+$EndComp
+$Comp
+L R R1
+U 1 1 5C7E0719
+P 10250 3750
+F 0 "R1" V 10330 3750 50  0000 C CNN
+F 1 "4k7" V 10400 3750 50  0000 C CNN
+F 2 "Resistors_SMD:R_0603" V 10180 3750 50  0001 C CNN
+F 3 "" H 10250 3750 50  0001 C CNN
+	1    10250 3750
+	-1   0    0    1
+$EndComp
+Wire Wire Line
+	10350 3600 10350 3550
+Wire Wire Line
+	10250 3600 10250 3550
+Wire Wire Line
+	10250 3550 10350 3550
+Wire Wire Line
+	10350 4050 10350 3900
+Connection ~ 10350 4050
+Wire Wire Line
+	10250 3900 10250 3950
+Connection ~ 10250 3950
+$Comp
+L Antenna AE1
+U 1 1 5C7E14EE
+P 5150 7400
+F 0 "AE1" H 5075 7475 50  0000 R CNN
+F 1 "Antenna" H 5075 7400 50  0000 R CNN
+F 2 "homebrew:helical_antenna_915mhz_hole" H 5150 7400 50  0001 C CNN
+F 3 "" H 5150 7400 50  0001 C CNN
+	1    5150 7400
+	0    1    1    0
+$EndComp
+Wire Wire Line
+	4950 7400 4800 7400
 $EndSCHEMATC
