File: hardware/rfboard.sch (KiCad schematic (older format))
At the start: 24 parts, among them J1 10118194-0001LF, J2 Conn_01x10, J3 Conn_01x10, P2 CONN_01X03, P3 CONN_01X04, U1 SAMD21E18, U2 RFM69CW-915MHZ, U3 MIC5504-3.3YM5-T5, U4 74LVC1G125

Commit message: Hardware revision v1.4:
- Add solder mask dam between pads on processor, regulator, buffer, and USB port
- Move antenna to not interfere with RFM69
- Added strain relief holes for LED connector
- Move USB capacitors down slightly to aid in fixing USB port shorts
- Fixed labeling of 3v3 pin
Parts:
- H3: value HOLE -> STRAIN_RELIEF; footprint homebrew:MountingHole_2.7mm_M2.5 -> homebrew:3_pin_2.54mm_pitch_strain_relief
- J1: footprint 10118194-0001LF:FRAMATOME_10118194-0001LF -> homebrew:FRAMATOME_10118194-0001LF_fixed_bridges
Changed lines of the file:
@@
 F 0 "J1" H 1209 7571 50  0000 L BNN
 F 1 "10118194-0001LF" H 1199 7049 50  0000 L BNN
-F 2 "10118194-0001LF:FRAMATOME_10118194-0001LF" H 1500 7350 50  0001 L BNN
+F 2 "homebrew:FRAMATOME_10118194-0001LF_fixed_bridges" H 1500 7350 50  0001 L BNN
 F 3 "Amphenol" H 1500 7350 50  0001 L BNN
 F 4 "0.25 USD" H 1500 7350 50  0001 L BNN "Field4"
@@
 F 3 "" H 6100 7100 60  0001 C CNN
 	1    6100 7100
-	1    0    0    -1
-$EndComp
-$Comp
-L Homebrew:HOLE H3
-U 1 1 5A843B2A
-P 6100 7500
-F 0 "H3" H 6100 7370 60  0000 C CNN
-F 1 "HOLE" H 6100 7620 60  0000 C CNN
-F 2 "homebrew:MountingHole_2.7mm_M2.5" H 6100 7500 60  0001 C CNN
-F 3 "" H 6100 7500 60  0001 C CNN
-	1    6100 7500
 	1    0    0    -1
 $EndComp
@@
 	1    0    0    -1
 $EndComp
+$Comp
+L Homebrew:HOLE H3
+U 1 1 5D26F404
+P 2500 6350
+F 0 "H3" H 2609 6403 60  0000 L CNN
+F 1 "STRAIN_RELIEF" H 2609 6297 60  0000 L CNN
+F 2 "homebrew:3_pin_2.54mm_pitch_strain_relief" H 2500 6350 60  0001 C CNN
+F 3 "" H 2500 6350 60  0001 C CNN
+	1    2500 6350
+	1    0    0    -1
+$EndComp
